Commit message: Fix contact state for Gazebo 7.

File: catkin_ws/src/journey/urdf/quadrotor_base.urdf.xacro (robot description, xacro)
@@ -10,9 +10,4 @@
   <xacro:macro name="quadrotor_base_macro" params="sim_name">
     <link name="base_link">
-      <inertial>
-        <mass value="1.477" />
-        <origin xyz="0 0 0" />
-        <inertia ixx="0.01152" ixy="0.0" ixz="0.0" iyy="0.01152" iyz="0.0" izz="0.0218" />
-      </inertial>
       <visual>
         <origin xyz="0 0 0" rpy="0 0 0" />
@@ -21,5 +16,5 @@
         </geometry>
       </visual>
-      <collision name="quadrotor_base_collision">
+      <collision>
         <origin xyz="0 0 0" rpy="0 0 0" />
         <geometry>
@@ -28,4 +23,15 @@
       </collision>
     </link>
+    <link name="dummy_link">
+      <inertial>
+        <mass value="1.477" />
+        <origin xyz="0 0 0" />
+        <inertia ixx="0.01152" ixy="0.0" ixz="0.0" iyy="0.01152" iyz="0.0" izz="0.0218" />
+      </inertial>
+    </link>
+    <joint name="dummy_joint" type="fixed">
+      <parent link="base_link"/>
+      <child link="dummy_link"/>
+    </joint>
     <gazebo reference="base_link">
       <turnGravityOff>false</turnGravityOff>
